Commit message: Update Noetic

File: aubo_description/urdf/aubo_i7.urdf (robot description, URDF)
Before this commit: robot aubo_i7, 8 links, 7 joints
Links:
- link base_link: mass 1.23448927826401 -> 1.53902; geometry collision mesh filename=package://aubo_description/meshes/aubo_i7/collision/link0.S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; visual mesh filename=package://aubo_description/meshes/aubo_i7/visual/link0.DAE
- link foreArm_Link: mass 2.88724337413486 -> 2.854995; geometry collision mesh filename=package://aubo_description/meshes/aubo_i7/collision/link3.S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; visual mesh filename=package://aubo_description/meshes/aubo_i7/visual/link3.DAE
- link shoulder_Link: mass 9.88740003439705 -> 4.848581; geometry collision mesh filename=package://aubo_description/meshes/aubo_i7/collision/link1.S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; visual mesh filename=package://aubo_description/meshes/aubo_i7/visual/link1.DAE
- link upperArm_Link: mass 4.46934833776782 -> 10.741921; geometry collision mesh filename=package://aubo_description/meshes/aubo_i7/collision/link2.S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; visual mesh filename=package://aubo_description/meshes/aubo_i7/visual/link2.DAE
- link wrist1_Link: mass 0.579814564711146 -> 1.628022; geometry collision mesh filename=package://aubo_description/meshes/aubo_i7/collision/link4.S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; visual mesh filename=package://aubo_description/meshes/aubo_i7/visual/link4.DAE
- link wrist2_Link: mass 0.579814565182749 -> 1.628022; geometry collision mesh filename=package://aubo_description/meshes/aubo_i7/collision/link5.S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; visual mesh filename=package://aubo_description/meshes/aubo_i7/visual/link5.DAE
- link wrist3_Link: mass 0.136689987013058 -> 0.1978; geometry collision mesh filename=package://aubo_description/meshes/aubo_i7/collision/link6.S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; visual mesh filename=package://aubo_description/meshes/aubo_i7/visual/link6.DAE
Joints:
- removed joint foreArm_Joint
- removed joint shoulder_Joint
- removed joint upperArm_Joint
- removed joint wrist1_Joint
- removed joint wrist2_Joint
- removed joint wrist3_Joint
- added joint foreArm_joint: type revolute, parent upperArm_Link, child foreArm_Link, origin xyz=0.368 0 0 rpy=-3.1415926535897932384626433832795 0 0, axis 0 0 1, limit lower=-6.283185307179586476925286766559 upper=6.283185307179586476925286766559 effort=133 velocity=2.5964
- added joint shoulder_joint: type revolute, parent base_link, child shoulder_Link, origin xyz=0 0 0.122 rpy=0 0 3.1415926535897932384626433832795, axis 0 0 1, limit lower=-6.283185307179586476925286766559 upper=6.283185307179586476925286766559 effort=133 velocity=2.5964
- added joint upperArm_joint: type revolute, parent shoulder_Link, child upperArm_Link, origin xyz=0 0.1215 0 rpy=-1.5707963267948966192313216916398 -1.5707963267948966192313216916398 0, axis 0 0 1, limit lower=-6.283185307179586476925286766559 upper=6.283185307179586476925286766559 effort=133 velocity=2.5964
- added joint wrist1_joint: type revolute, parent foreArm_Link, child wrist1_Link, origin xyz=0.316 0 0 rpy=3.1415926535897932384626433832795 0 1.5707963267948966192313216916398, axis 0 0 1, limit lower=-6.283185307179586476925286766559 upper=6.283185307179586476925286766559 effort=13.5 velocity=3.1105
- added joint wrist2_joint: type revolute, parent wrist1_Link, child wrist2_Link, origin xyz=0 0.1025 0 rpy=-1.5707963267948966192313216916398 0 0, axis 0 0 1, limit lower=-6.283185307179586476925286766559 upper=6.283185307179586476925286766559 effort=13.5 velocity=3.1105
- added joint wrist3_joint: type revolute, parent wrist2_Link, child wrist3_Link, origin xyz=0 -0.094 0 rpy=1.5707963267948966192313216916398 0 1.7907E-15, axis 0 0 1, limit lower=-6.283185307179586476925286766559 upper=6.283185307179586476925286766559 effort=13.5 velocity=3.1105
